File: macro-pad-1.kicad_pcb (KiCad board)
At the start: 2 copper layers, 93.9 x 38.1 mm, 24 parts, among them SW1 SW_Push, U1 ATmega32U4-AU, Y1 Crystal_GND24_Small

Commit message: PCB routing, not done
Parts:
- F1, R3, R4, SW1, USB1: moved to B.Cu
- moved R4 44.0 mm to (72.5, 80.1), turned to 90 degrees
- moved SW1 42.9 mm to (74.5, 98.8), turned to 180 degrees
- moved R3 40.1 mm to (74.8, 80.1), turned to 90 degrees
- moved R2 37.0 mm to (112.9, 93.8)
- moved F1 32.3 mm to (69.1, 85.3), turned to 90 degrees
- moved R1 28.6 mm to (88.6, 80.8), turned to 90 degrees
- moved C1 24.0 mm to (107.2, 77.0), turned to 90 degrees
- moved C4 23.5 mm to (91.8, 80.7), turned to 270 degrees
- moved C2 23.3 mm to (98.3, 77.0), turned to 270 degrees
- moved C5 23.0 mm to (113.0, 83.8), turned to 90 degrees
- moved Y1 21.8 mm to (102.5, 77.0), turned to 180 degrees
- moved C6 21.7 mm to (107.6, 97.4)
- moved C7 20.9 mm to (97.9, 97.4), turned to 0 degrees
- moved C3 20.2 mm to (92.0, 85.7), turned to 0 degrees
- moved USB1 14.7 mm to (74.0, 69.8), turned to 270 degrees
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Routing:
- net GND: track 0.00 -> 99.4 mm
- net +5V: track 0.00 -> 61.6 mm, vias 0 -> 2
- net Net-(R2-Pad1): track 0.00 -> 45.7 mm, vias 0 -> 4
- net Net-(R4-Pad1): track 0.00 -> 29.0 mm
- net Net-(R3-Pad1): track 0.00 -> 26.4 mm
- net Net-(D3-Pad2): track 0.00 -> 18.4 mm
- net VCC: track 0.00 -> 11.8 mm
- net Net-(C3-Pad1): track 0.00 -> 8.45 mm, vias 0 -> 2
- net Net-(C1-Pad1): track 0.00 -> 8.25 mm
- net D+: track 0.00 -> 5.28 mm
- net D-: track 0.00 -> 5.16 mm
Other:
- outline, holes or cut-outs redrawn
- net class Default: trace_width 0.25 -> 0.254
- net class Power added: clearance 0.2, trace_width 0.381, via_dia 0.8, via_drill 0.4
